Commit message: Change jib to JIB in v5 urdf

File: urdf/altas_v5.urdf (robot description, URDF)
Before this commit: robot drc_skeleton, 37 links, 36 joints
Links:
- link l_clav: geometry collision mesh filename=package://JIB/meshes_unplugged/l_clav.dae; visual mesh filename=package://JIB/meshes_unplugged/l_clav.dae
- link l_foot: geometry collision mesh filename=package://JIB/meshes_unplugged/l_foot.dae; visual mesh filename=package://JIB/meshes_unplugged/l_foot.dae
- link l_larm: geometry collision mesh filename=package://JIB/meshes_unplugged/l_larm.dae; visual mesh filename=package://JIB/meshes_unplugged/l_larm.dae
- link l_lfarm: geometry collision mesh filename=package://JIB/meshes_unplugged/l_hand.dae; visual mesh filename=package://JIB/meshes_unplugged/l_hand.dae
- link l_lglut: geometry collision mesh filename=package://JIB/meshes_unplugged/l_lglut.dae; visual mesh filename=package://JIB/meshes_unplugged/l_lglut.dae
- link l_lleg: geometry collision mesh filename=package://JIB/meshes_unplugged/l_lleg.dae; visual mesh filename=package://JIB/meshes_unplugged/l_lleg.dae
- link l_scap: geometry collision mesh filename=package://JIB/meshes_unplugged/l_scap.dae; visual mesh filename=package://JIB/meshes_unplugged/l_scap.dae
- link l_talus: geometry collision mesh filename=package://JIB/meshes_unplugged/l_talus.dae; visual mesh filename=package://JIB/meshes_unplugged/l_talus.dae
- link l_uarm: geometry collision mesh filename=package://JIB/meshes_unplugged/l_uarm.dae; visual mesh filename=package://JIB/meshes_unplugged/l_uarm.dae
- link l_ufarm: geometry collision mesh filename=package://JIB/meshes_unplugged/l_farm.dae; visual mesh filename=package://JIB/meshes_unplugged/l_farm.dae
- link l_uglut: geometry collision mesh filename=package://JIB/meshes_unplugged/l_uglut.dae; visual mesh filename=package://JIB/meshes_unplugged/l_uglut.dae
- link l_uleg: geometry collision mesh filename=package://JIB/meshes_unplugged/l_uleg.dae; visual mesh filename=package://JIB/meshes_unplugged/l_uleg.dae
- link ltorso: geometry collision mesh filename=package://JIB/meshes_unplugged/ltorso.dae; visual mesh filename=package://JIB/meshes_unplugged/ltorso.dae
- link mtorso: geometry collision mesh filename=package://JIB/meshes_unplugged/mtorso.dae; visual mesh filename=package://JIB/meshes_unplugged/mtorso.dae
- link pelvis: geometry collision mesh filename=package://JIB/meshes_unplugged/pelvis.dae; visual mesh filename=package://JIB/meshes_unplugged/pelvis.dae
- link r_clav: geometry collision mesh filename=package://JIB/meshes_unplugged/r_clav.dae; visual mesh filename=package://JIB/meshes_unplugged/r_clav.dae
- link r_foot: geometry collision mesh filename=package://JIB/meshes_unplugged/r_foot.dae; visual mesh filename=package://JIB/meshes_unplugged/r_foot.dae
- link r_larm: geometry collision mesh filename=package://JIB/meshes_unplugged/r_larm.dae; visual mesh filename=package://JIB/meshes_unplugged/r_larm.dae
- link r_lfarm: geometry collision mesh filename=package://JIB/meshes_unplugged/r_hand.dae; visual mesh filename=package://JIB/meshes_unplugged/r_hand.dae
- link r_lglut: geometry collision mesh filename=package://JIB/meshes_unplugged/r_lglut.dae; visual mesh filename=package://JIB/meshes_unplugged/r_lglut.dae
- link r_lleg: geometry collision mesh filename=package://JIB/meshes_unplugged/r_lleg.dae; visual mesh filename=package://JIB/meshes_unplugged/r_lleg.dae
- link r_scap: geometry collision mesh filename=package://JIB/meshes_unplugged/r_scap.dae; visual mesh filename=package://JIB/meshes_unplugged/r_scap.dae
- link r_talus: geometry collision mesh filename=package://JIB/meshes_unplugged/r_talus.dae; visual mesh filename=package://JIB/meshes_unplugged/r_talus.dae
- link r_uarm: geometry collision mesh filename=package://JIB/meshes_unplugged/r_uarm.dae; visual mesh filename=package://JIB/meshes_unplugged/r_uarm.dae
- link r_ufarm: geometry collision mesh filename=package://JIB/meshes_unplugged/r_farm.dae; visual mesh filename=package://JIB/meshes_unplugged/r_farm.dae
- link r_uglut: geometry collision mesh filename=package://JIB/meshes_unplugged/r_uglut.dae; visual mesh filename=package://JIB/meshes_unplugged/r_uglut.dae
- link r_uleg: geometry collision mesh filename=package://JIB/meshes_unplugged/r_uleg.dae; visual mesh filename=package://JIB/meshes_unplugged/r_uleg.dae
- link utorso: geometry collision mesh filename=package://JIB/meshes_unplugged/utorso.dae; visual mesh filename=package://JIB/meshes_unplugged/utorso.dae
